Commit message: Primer commit

File: agro_description/urdf/agro2.urdf.xacro (robot description, xacro)
@@ -5,5 +5,5 @@
             <origin xyz="0.0 0.0 0.0" rpy="0.0 0.0 0.0"/>
             <geometry>
-                <box size="0.4 0.2 0.3"/>
+                <box size="0.5 0.316 0.16"/>
             </geometry>
             <material name="">
@@ -17,5 +17,5 @@
             <origin xyz="0.0 0.0 0.0" rpy="1.57 0.0 0.0"/>
             <geometry>
-                <cylinder radius="0.3" length="0.1"/>
+                <cylinder radius="0.12" length="0.0615"/>
             </geometry>
             <material name="">
