Commit message: modelo2

File: agro_description/urdf/agro.urdf.xacro (robot description, xacro)
@@ -29,5 +29,5 @@
         <parent link="base_link"/>
         <child link="wheel_1"/>
-        <axis xyz="0.0 0.0 1.0"/>
+        <axis xyz="0.0 1.0 0.0"/>
         <limit lower="0.0" upper="0.0" effort="0.0" velocity="0.0"/>
     </joint>

File: agro_description/urdf/agro2.urdf.xacro (robot description, xacro)
@@ -1,4 +1,10 @@
 <?xml version="1.0"?>
 <robot xmlns:xacro="http://www.ros.org/wiki/xacro" name="robot_name">
+  <!-- ************************ -->
+  <!--  variables -->
+  <!-- ************************ -->
+  <!--<xacro:property name="wheel_radius" value="0.0615"/>
+  <xacro:property name="base_width" value="0.316"/>
+  <xacro:property name="wheel_distance" value="0.225"/>-->
     <link name="base_link">
         <visual>
@@ -13,5 +19,6 @@
         </visual>
     </link>
-    <link name="wheel_1">
+    <xacro:macro name="wheel_link" params="prefix">
+     <link name="${prefix}_wheel">
         <visual name="">
             <origin xyz="0.0 0.0 0.0" rpy="1.57 0.0 0.0"/>
@@ -24,11 +31,22 @@
             </material>
         </visual>
-    </link>
-    <joint name="base_wheel_1_joint" type="continuous">
-        <origin xyz="0.5 0.4 -0.2" rpy="0.0 0.0 0.0"/>
+     </link>
+    </xacro:macro>
+    <xacro:wheel_link prefix="front_left" />
+    <xacro:wheel_link prefix="front_right" />
+    <xacro:wheel_link prefix="near_left" />
+    <xacro:wheel_link prefix="near_right" />
+    <xacro:macro name="wheel_joint" params="prefix x y">
+     <joint name="${prefix}_joint" type="continuous">
+        <origin xyz="${x} ${y} 0.0" rpy="0.0 0.0 0.0"/>
         <parent link="base_link"/>
-        <child link="wheel_1"/>
-        <axis xyz="0.0 0.0 1.0"/>
+        <child link="${prefix}_wheel"/>
+        <axis xyz="0.0 0.1 0.0"/>
         <limit lower="0.0" upper="0.0" effort="0.0" velocity="0.0"/>
-    </joint>
+     </joint>
+    </xacro:macro>
+    <xacro:wheel_joint prefix="front_left" x="0.225" y="${(0.0615 + 0.316)/2}" />
+    <xacro:wheel_joint prefix="front_right" x="0.225" y="${-(0.0615 + 0.316)/2}" />
+    <xacro:wheel_joint prefix="near_left" x="-0.225" y="${(0.0615 + 0.316)/2}" />
+    <xacro:wheel_joint prefix="near_right" x="-0.225" y="${-(0.0615 + 0.316)/2}" />
 </robot>

Commit message: Trabajadno en agro_description

File: agro_description/urdf/agro.urdf.xacro (robot description, xacro)
@@ -1,34 +1,51 @@
 <?xml version="1.0"?>
 <robot xmlns:xacro="http://www.ros.org/wiki/xacro" name="robot_name">
+  <!-- ************************ -->
+  <!--  variables -->
+  <!-- ************************ -->
+  <!--<xacro:property name="wheel_radius" value="0.0615"/>
+  <xacro:property name="base_width" value="0.316"/>
+  <xacro:property name="wheel_distance" value="0.225"/>-->
+    <xacro:include filename="$(find agro_description)/urdf/xacro/wheel.xacro"/>
+     <!-- Base-->
     <link name="base_link">
         <visual>
             <origin xyz="0.0 0.0 0.0" rpy="0.0 0.0 0.0"/>
             <geometry>
-                <box size="0.4 0.2 0.3"/>
+                <!--box size="0.5 0.316 0.16"/-->
+                <mesh filename="file://$(find agro_description)/mesh/base.stl" scale="0.001 0.001 0.001"/>
             </geometry>
-            <material name="">
-                <color rgba="1.0 0.0 0.0 1.0"/>
-                <texture filename=""/>
+            <material name="wood">
+                <color rgba="0.76 0.60 0.42 1.0"/> <!-- Color madera -->
             </material>
         </visual>
     </link>
-    <link name="wheel_1">
-        <visual name="">
-            <origin xyz="0.0 0.0 0.0" rpy="1.57 0.0 0.0"/>
+    <!-- Chassis-->
+    <link name="chassis_link">
+        <visual>
+            <origin xyz="0.0 0.0 0.0" rpy="0.0 0.0 0.0"/>
             <geometry>
-                <cylinder radius="0.3" length="0.1"/>
+                <!--box size="0.5 0.316 0.16"/-->
+                <mesh filename="file://$(find agro_description)/mesh/chassis.stl" scale="0.001 0.001 0.001"/>
             </geometry>
-            <material name="">
-                <color rgba="1.0 0.0 0.0 1.0"/>
-                <texture filename=""/>
+            <material name="steel">
+                <color rgba="0.70 0.70 0.70 1.0"/> <!-- Color acero -->
             </material>
         </visual>
     </link>
-    <joint name="base_wheel_1_joint" type="continuous">
-        <origin xyz="0.5 0.4 -0.2" rpy="0.0 0.0 0.0"/>
+    <joint name="base_chassis_joint" type="fixed">
+        <origin xyz="0.0 0.0 0.0" rpy="0.0 0.0 0.0"/>
         <parent link="base_link"/>
-        <child link="wheel_1"/>
-        <axis xyz="0.0 1.0 0.0"/>
-        <limit lower="0.0" upper="0.0" effort="0.0" velocity="0.0"/>
+        <child link="chassis_link"/>
     </joint>
+    <!-- Wheels-->
+    <xacro:wheel_link prefix="front_left" />
+    <xacro:wheel_link prefix="front_right" />
+    <xacro:wheel_link prefix="near_left" />
+    <xacro:wheel_link prefix="near_right" />
+    <xacro:wheel_joint prefix="front_left" x="0.210" y="0.224" z="-0.1376"/>
+    <xacro:wheel_joint prefix="front_right" x="0.210" y="-0.224" z="-0.1376"/>
+    <xacro:wheel_joint prefix="near_left" x="-0.210" y="0.224" z="-0.1376"/>
+    <xacro:wheel_joint prefix="near_right" x="-0.219" y="-0.224" z="-0.1376"/>
+    <!-- Base camera-->
 </robot>

Commit message: robot completo

File: agro_description/urdf/agro.urdf.xacro (robot description, xacro)
@@ -39,4 +39,40 @@
         <child link="chassis_link"/>
     </joint>
+    <!-- soporte-->
+    <link name="soporte_link">
+        <visual>
+            <origin xyz="0.0 0.0 0.0" rpy="0.0 0.0 0.0"/>
+            <geometry>
+                <!--box size="0.5 0.316 0.16"/-->
+                <mesh filename="file://$(find agro_description)/mesh/soporte.stl" scale="0.001 0.001 0.001"/>
+            </geometry>
+            <material name="steel">
+                <color rgba="0.70 0.70 0.70 1.0"/> <!-- Color acero -->
+            </material>
+        </visual>
+    </link>
+    <joint name="base_soporte_joint" type="fixed">
+        <origin xyz="0.21 0.0 0.16" rpy="0.0 0.0 0.0"/>
+        <parent link="base_link"/>
+        <child link="soporte_link"/>
+    </joint>
+    <!-- base_camara-->
+    <link name="base_camara_link">
+        <visual>
+            <origin xyz="0.0 0.0 0.0" rpy="0.0 0.0 0.0"/>
+            <geometry>
+                <!--box size="0.5 0.316 0.16"/-->
+                <mesh filename="file://$(find agro_description)/mesh/base_camara.stl" scale="0.001 0.001 0.001"/>
+            </geometry>
+            <material name="steel">
+                <color rgba="0.76 0.60 0.42 1.0"/> <!-- Color madera -->
+            </material>
+        </visual>
+    </link>
+    <joint name="base_camara_joint" type="fixed">
+        <origin xyz="0.21 0.0 0.76" rpy="0.0 0.0 0.0"/>
+        <parent link="base_link"/>
+        <child link="base_camara_link"/>
+    </joint>
     <!-- Wheels-->
     <xacro:wheel_link prefix="front_left" />

Commit message: Test gazebo

File: agro_description/urdf/agro.urdf.xacro (robot description, xacro)
@@ -8,4 +8,5 @@
   <xacro:property name="wheel_distance" value="0.225"/>-->
     <xacro:include filename="$(find agro_description)/urdf/xacro/wheel.xacro"/>
+    <xacro:include filename="$(find agro_description)/urdf/xacro/gazebo.xacro"/>
      <!-- Base-->
     <link name="base_link">
@@ -20,4 +21,13 @@
             </material>
         </visual>
+        <xacro:inertial_box mass="${base_mass}" x="${base_altura}" y="${base_largo}" z="${base_ancho}">
+            <origin xyz="0.0 0.0 0.0" rpy="0.0 0.0 0.0"/>
+        </xacro:inertial_box>
+        <collision>
+            <origin xyz="0.0 0.0 0.0" rpy="0.0 0.0 0.0"/>
+            <geometry>
+                <box size="${base_altura} ${base_largo} ${base_ancho}"/>
+            </geometry>
+        </collision>
     </link>
     <!-- Chassis-->
@@ -33,4 +43,13 @@
             </material>
         </visual>
+        <xacro:inertial_box mass="${chassis_mass}" x="${chassis_altura}" y="${chassis_largo}" z="${chassis_ancho}">
+            <origin xyz="0.0 0.0 0.0" rpy="0.0 0.0 0.0"/>
+        </xacro:inertial_box>
+        <collision>
+            <origin xyz="0.0 0.0 0.0" rpy="0.0 0.0 0.0"/>
+            <geometry>
+                <box size="${chassis_altura} ${chassis_largo} ${chassis_ancho}"/>
+            </geometry>
+        </collision>
     </link>
     <joint name="base_chassis_joint" type="fixed">
@@ -40,13 +59,12 @@
     </joint>
     <!-- soporte-->
-    <link name="soporte_link">
+    <!--link name="soporte_link">
         <visual>
             <origin xyz="0.0 0.0 0.0" rpy="0.0 0.0 0.0"/>
             <geometry>
-                <!--box size="0.5 0.316 0.16"/-->
                 <mesh filename="file://$(find agro_description)/mesh/soporte.stl" scale="0.001 0.001 0.001"/>
             </geometry>
             <material name="steel">
-                <color rgba="0.70 0.70 0.70 1.0"/> <!-- Color acero -->
+                <color rgba="0.70 0.70 0.70 1.0"/>
             </material>
         </visual>
@@ -56,15 +74,32 @@
         <parent link="base_link"/>
         <child link="soporte_link"/>
-    </joint>
-    <!-- base_camara-->
-    <link name="base_camara_link">
+    </joint-->
+    <!-- soporte-->
+    <!--link name="soporte_link">
         <visual>
             <origin xyz="0.0 0.0 0.0" rpy="0.0 0.0 0.0"/>
             <geometry>
-                <!--box size="0.5 0.316 0.16"/-->
+                <box size="0.5 0.316 0.16"/>
+                <mesh filename="file://$(find agro_description)/mesh/soporte.stl" scale="0.001 0.001 0.001"/>
+            </geometry>
+            <material name="steel">
+                <color rgba="0.70 0.70 0.70 1.0"/>
+            </material>
+        </visual>
+    </link>
+    <joint name="base_soporte_joint" type="fixed">
+        <origin xyz="0.21 0.0 0.16" rpy="0.0 0.0 0.0"/>
+        <parent link="base_link"/>
+        <child link="soporte_link"/>
+    </joint-->
+    <!-- base_camara-->
+    <!--link name="base_camara_link">
+        <visual>
+            <origin xyz="0.0 0.0 0.0" rpy="0.0 0.0 0.0"/>
+            <geometry>
                 <mesh filename="file://$(find agro_description)/mesh/base_camara.stl" scale="0.001 0.001 0.001"/>
             </geometry>
             <material name="steel">
-                <color rgba="0.76 0.60 0.42 1.0"/> <!-- Color madera -->
+                <color rgba="0.76 0.60 0.42 1.0"/>
             </material>
         </visual>
@@ -74,5 +109,5 @@
         <parent link="base_link"/>
         <child link="base_camara_link"/>
-    </joint>
+    </joint-->
     <!-- Wheels-->
     <xacro:wheel_link prefix="front_left" />
@@ -84,4 +119,4 @@
     <xacro:wheel_joint prefix="near_left" x="-0.210" y="0.224" z="-0.1376"/>
     <xacro:wheel_joint prefix="near_right" x="-0.219" y="-0.224" z="-0.1376"/>
-    <!-- Base camera-->
+    <xacro:ros2_control/>
 </robot>

File: agro_description/urdf/xacro/wheel.xacro (robot description, xacro)
@@ -15,8 +15,8 @@
         </visual>
         <xacro:inertial_cylinder mass="${wheel_mass}" length="${wheel_length}" radius="${wheel_radius}">
-            <origin xyz="0.0 0 0" rpy="0 0 0"/>
+            <origin xyz="0.0 0 0" rpy="1.57  0 0"/>
         </xacro:inertial_cylinder>
         <collision>
-            <origin xyz="0.0 0.0 0.0" rpy="0.0 0.0 0.0"/>
+            <origin xyz="0.0 0.0 0.0" rpy="1.57  0.0 0.0"/>
             <geometry>
                 <cylinder radius="${wheel_radius}" length="${wheel_length}"/>
@@ -30,6 +30,7 @@
         <parent link="base_link"/>
         <child link="${prefix}_wheel"/>
-        <axis xyz="0.0 0.1 0.0"/>
-        <limit lower="0.0" upper="0.0" effort="0.0" velocity="0.0"/>
+        <axis xyz="0.0 1.0 0.0"/>
+        <limit effort="1.5" velocity="30.0" />
+        <dynamics damping="0.001" friction="0.001" />
      </joint>
     </xacro:macro>

Commit message: inercia y colision

File: agro_description/urdf/agro.urdf.xacro (robot description, xacro)
@@ -4,7 +4,4 @@
   <!--  variables -->
   <!-- ************************ -->
-  <!--<xacro:property name="wheel_radius" value="0.0615"/>
-  <xacro:property name="base_width" value="0.316"/>
-  <xacro:property name="wheel_distance" value="0.225"/>-->
     <xacro:include filename="$(find agro_description)/urdf/xacro/wheel.xacro"/>
     <xacro:include filename="$(find agro_description)/urdf/xacro/gazebo.xacro"/>
@@ -21,11 +18,11 @@
             </material>
         </visual>
-        <xacro:inertial_box mass="${base_mass}" x="${base_altura}" y="${base_largo}" z="${base_ancho}">
-            <origin xyz="0.0 0.0 0.0" rpy="0.0 0.0 0.0"/>
+        <xacro:inertial_box mass="${base_mass}" x="${base_largo}" y="${base_ancho}" z="${base_altura}">
+            <origin xyz="0.0 0.0 ${(base_altura)/2}" rpy="0.0 0.0 0.0"/>
         </xacro:inertial_box>
         <collision>
-            <origin xyz="0.0 0.0 0.0" rpy="0.0 0.0 0.0"/>
+            <origin xyz="0.0 0.0 ${(base_altura)/2}" rpy="0.0 0.0 0.0"/>
             <geometry>
-                <box size="${base_altura} ${base_largo} ${base_ancho}"/>
+                <box size="${base_largo} ${base_ancho} ${base_altura}"/>   <!--0.5 0.316 0.16-->
             </geometry>
         </collision>
@@ -43,11 +40,11 @@
             </material>
         </visual>
-        <xacro:inertial_box mass="${chassis_mass}" x="${chassis_altura}" y="${chassis_largo}" z="${chassis_ancho}">
-            <origin xyz="0.0 0.0 0.0" rpy="0.0 0.0 0.0"/>
+        <xacro:inertial_box mass="${chassis_mass}" x="${chassis_largo}" y="${chassis_ancho}" z="${chassis_altura}">
+            <origin xyz="0.0 0.0 ${-(chassis_altura)/2}" rpy="0.0 0.0 0.0"/>
         </xacro:inertial_box>
         <collision>
-            <origin xyz="0.0 0.0 0.0" rpy="0.0 0.0 0.0"/>
+            <origin xyz="0.0 0.0 ${-(chassis_altura)/2}" rpy="0.0 0.0 0.0"/>
             <geometry>
-                <box size="${chassis_altura} ${chassis_largo} ${chassis_ancho}"/>
+                <box size="${chassis_largo} ${chassis_ancho} ${chassis_altura}"/>
             </geometry>
         </collision>
@@ -58,6 +55,6 @@
         <child link="chassis_link"/>
     </joint>
-    <!-- soporte-->
-    <!--link name="soporte_link">
+    <!-- soporte -->
+    <link name="soporte_link">
         <visual>
             <origin xyz="0.0 0.0 0.0" rpy="0.0 0.0 0.0"/>
@@ -69,4 +66,13 @@
             </material>
         </visual>
+        <xacro:inertial_box mass="${soporte_mass}" x="${soporte_largo}" y="${soporte_ancho}" z="${soporte_altura}">
+            <origin xyz="0.0 0.0 0.30" rpy="0.0 0.0 0.0"/>
+        </xacro:inertial_box>
+        <collision>
+            <origin xyz="0.0 0.0 0.30" rpy="0.0 0.0 0.0"/>
+            <geometry>
+                <box size="${soporte_largo} ${soporte_ancho} ${soporte_altura}"/>
+            </geometry>
+        </collision>
     </link>
     <joint name="base_soporte_joint" type="fixed">
@@ -74,25 +80,7 @@
         <parent link="base_link"/>
         <child link="soporte_link"/>
-    </joint-->
-    <!-- soporte-->
-    <!--link name="soporte_link">
-        <visual>
-            <origin xyz="0.0 0.0 0.0" rpy="0.0 0.0 0.0"/>
-            <geometry>
-                <box size="0.5 0.316 0.16"/>
-                <mesh filename="file://$(find agro_description)/mesh/soporte.stl" scale="0.001 0.001 0.001"/>
-            </geometry>
-            <material name="steel">
-                <color rgba="0.70 0.70 0.70 1.0"/>
-            </material>
-        </visual>
-    </link>
-    <joint name="base_soporte_joint" type="fixed">
-        <origin xyz="0.21 0.0 0.16" rpy="0.0 0.0 0.0"/>
-        <parent link="base_link"/>
-        <child link="soporte_link"/>
-    </joint-->
+    </joint>
     <!-- base_camara-->
-    <!--link name="base_camara_link">
+    <link name="base_camara_link">
         <visual>
             <origin xyz="0.0 0.0 0.0" rpy="0.0 0.0 0.0"/>
@@ -100,8 +88,17 @@
                 <mesh filename="file://$(find agro_description)/mesh/base_camara.stl" scale="0.001 0.001 0.001"/>
             </geometry>
-            <material name="steel">
-                <color rgba="0.76 0.60 0.42 1.0"/>
+            <material name="wood">
+                <color rgba="0.76 0.60 0.42 1.0"/> <!-- Color madera -->
             </material>
         </visual>
+        <xacro:inertial_box mass="${base_camara_mass}" x="${base_camara_largo}" y="${base_camara_ancho}" z="${base_camara_altura}">
+            <origin xyz="0.01 0.0 0.0015" rpy="0.0 0.0 0.0"/>
+        </xacro:inertial_box>
+        <collision>
+            <origin xyz="0.01 0.0 0.0015" rpy="0.0 0.0 0.0"/>
+            <geometry>
+                <box size="${base_camara_largo} ${base_camara_ancho} ${base_camara_altura}"/>
+            </geometry>
+        </collision>
     </link>
     <joint name="base_camara_joint" type="fixed">
@@ -109,5 +106,5 @@
         <parent link="base_link"/>
         <child link="base_camara_link"/>
-    </joint-->
+    </joint>
     <!-- Wheels-->
     <xacro:wheel_link prefix="front_left" />

File: agro_description/urdf/xacro/properties.xacro (robot description, xacro)
@@ -2,14 +2,22 @@
 <robot xmlns:xacro="http://www.ros.org/wiki/xacro" >
     <!-- sizes-->
-    <xacro:property name="wheel_radius" value="0.12" />
+    <xacro:property name="wheel_radius" value="0.0601" />
     <xacro:property name="wheel_length" value="0.0615" />
     <xacro:property name="wheel_mass" value="0.2" />
     <xacro:property name="base_altura" value="0.16" />
     <xacro:property name="base_largo" value="0.5" />
-    <xacro:property name="base_ancho" value="0.316" />
+    <xacro:property name="base_ancho" value="0.320" />
     <xacro:property name="base_mass" value="0.2" />
-    <xacro:property name="chassis_altura" value="0.2" />
-    <xacro:property name="chassis_largo" value="0.2" />
-    <xacro:property name="chassis_ancho" value="0.2" />
+    <xacro:property name="chassis_altura" value="0.1596" />
+    <xacro:property name="chassis_largo" value="0.46" />
+    <xacro:property name="chassis_ancho" value="0.44" />
     <xacro:property name="chassis_mass" value="0.2" />
+    <xacro:property name="soporte_altura" value="0.6" />
+    <xacro:property name="soporte_largo" value="0.02" />
+    <xacro:property name="soporte_ancho" value="0.02" />
+    <xacro:property name="soporte_mass" value="0.1" />
+    <xacro:property name="base_camara_altura" value="0.003" />
+    <xacro:property name="base_camara_largo" value="0.16" />
+    <xacro:property name="base_camara_ancho" value="0.15" />
+    <xacro:property name="base_camara_mass" value="0.05" />
 </robot>

Commit message: COnfigurando ekf

File: agro_description/urdf/agro.urdf.xacro (robot description, xacro)
@@ -117,3 +117,4 @@
     <xacro:wheel_joint prefix="near_right" x="-0.219" y="-0.224" z="-0.1376"/>
     <xacro:ros2_control/>
+    <xacro:plugins_gazebo/>
 </robot>

File: agro_description/urdf/xacro/gazebo.xacro (robot description, xacro)
@@ -27,3 +27,38 @@
         </ros2_control>
   </xacro:macro>
+  <xacro:macro name="plugins_gazebo">
+    <gazebo reference="base_link">
+        <sensor name="tb3_gps" type="navsat">
+          <always_on>true</always_on>
+          <update_rate>1</update_rate>
+          <pose>0 0 0 0 0 0</pose>
+          <!--gps>
+            <position_sensing>
+              <horizontal>
+                <noise type="gaussian">
+                  <mean>0.0</mean>
+                  <stddev>0.01</stddev>
+                </noise>
+              </horizontal>
+              <vertical>
+                <noise type="gaussian">
+                  <mean>0.0</mean>
+                  <stddev>0.01</stddev>
+                </noise>
+              </vertical>
+            </position_sensing>
+          </gps-->
+           <topic>gps/fix</topic>
+        </sensor>
+    </gazebo>
+    <gazebo reference="base_link">
+      <sensor name="imu_sensor" type="imu">
+          <always_on>1</always_on>
+          <update_rate>1</update_rate>
+          <visualize>true</visualize>
+          <topic>imu</topic>
+          <frame_id>base_link</frame_id>
+      </sensor>
+    </gazebo>
+  </xacro:macro>
 </robot>
