Commit message: ekf funcionando

File: agro_description/urdf/agro.urdf.xacro (robot description, xacro)
@@ -6,4 +6,6 @@
     <xacro:include filename="$(find agro_description)/urdf/xacro/wheel.xacro"/>
     <xacro:include filename="$(find agro_description)/urdf/xacro/gazebo.xacro"/>
+    <link name= "base_footprint">
+    </link>
      <!-- Base-->
     <link name="base_link">
@@ -28,4 +30,9 @@
         </collision>
     </link>
+    <joint name="base_footprint_joint" type="fixed">
+        <origin xyz="0.0 0.0 0.2" rpy="0.0 0.0 0.0"/>
+        <parent link="base_footprint"/>
+        <child link="base_link"/>
+    </joint>
     <!-- Chassis-->
     <link name="chassis_link">
@@ -116,4 +123,30 @@
     <xacro:wheel_joint prefix="near_left" x="-0.210" y="0.224" z="-0.1376"/>
     <xacro:wheel_joint prefix="near_right" x="-0.219" y="-0.224" z="-0.1376"/>
+    <!-- soporte -->
+    <link name="robot_agro/base_footprint/imu_sensor">
+        <visual>
+            <origin xyz="0.0 0.0 0.0" rpy="0.0 0.0 0.0"/>
+            <geometry>
+                <mesh filename="file://$(find agro_description)/mesh/soporte.stl" scale="0.001 0.001 0.001"/>
+            </geometry>
+            <material name="steel">
+                <color rgba="0.70 0.70 0.70 1.0"/>
+            </material>
+        </visual>
+        <xacro:inertial_box mass="${soporte_mass}" x="${soporte_largo}" y="${soporte_ancho}" z="${soporte_altura}">
+            <origin xyz="0.0 0.0 0.30" rpy="0.0 0.0 0.0"/>
+        </xacro:inertial_box>
+        <collision>
+            <origin xyz="0.0 0.0 0.30" rpy="0.0 0.0 0.0"/>
+            <geometry>
+                <box size="${soporte_largo} ${soporte_ancho} ${soporte_altura}"/>
+            </geometry>
+        </collision>
+    </link>
+    <joint name="base_imu_joint" type="fixed">
+        <origin xyz="0.21 0.0 0.16" rpy="0.0 0.0 0.0"/>
+        <parent link="base_footprint"/>
+        <child link="robot_agro/base_footprint/imu_sensor"/>
+    </joint>
     <xacro:ros2_control/>
     <xacro:plugins_gazebo/>

File: agro_description/urdf/xacro/gazebo.xacro (robot description, xacro)
@@ -25,4 +25,16 @@
             <xacro:ros2_control wheel="near_left"/>
             <xacro:ros2_control wheel="near_right"/>
+            <sensor name="imu">
+              <state_interface name="orientation.x" />
+              <state_interface name="orientation.y" />
+              <state_interface name="orientation.z" />
+              <state_interface name="orientation.w" />
+              <state_interface name="angular_velocity.x" />
+              <state_interface name="angular_velocity.y" />
+              <state_interface name="angular_velocity.z" />
+              <state_interface name="linear_acceleration.x" />
+              <state_interface name="linear_acceleration.y" />
+              <state_interface name="linear_acceleration.z" />
+            </sensor>
         </ros2_control>
   </xacro:macro>
@@ -52,11 +64,49 @@
         </sensor>
     </gazebo>
+    <!-- Gauss noise macro -->
+    <xacro:macro name="gauss_noise"
+      params="mean:=0.0 stddev:=0.0 bias_mean:=0.0 bias_stddev:=0.0 precision:=0.0">
+      <noise type="gaussian">
+        <mean>${mean}</mean>
+        <stddev>${stddev}</stddev>
+        <bias_mean>${bias_mean}</bias_mean>
+        <bias_stddev>${bias_stddev}</bias_stddev>
+        <precision>${precision}</precision>
+      </noise>
+    </xacro:macro>
     <gazebo reference="base_link">
       <sensor name="imu_sensor" type="imu">
-          <always_on>1</always_on>
-          <update_rate>50</update_rate>
-          <visualize>true</visualize>
-          <topic>imu</topic>
-          <frame_id>base_link</frame_id>
+        <always_on>true</always_on>
+        <update_rate>20</update_rate>
+        <topic>imu</topic>
+        <visualize>false</visualize>
+        <enable_metrics>false</enable_metrics>
+        <frame_id>base_link</frame_id>
+        <imu>
+          <angular_velocity>
+            <!-- rad/s | no bias_mean in datasheet -->
+            <x>
+              <xacro:gauss_noise stddev="5.24e-3" bias_mean="2.0e-3" precision="1.07e-3" />
+            </x>
+            <y>
+              <xacro:gauss_noise stddev="5.24e-3" bias_mean="2.0e-3" precision="1.07e-3" />
+            </y>
+            <z>
+              <xacro:gauss_noise stddev="5.24e-3" bias_mean="2.0e-3" precision="1.07e-3" />
+            </z>
+          </angular_velocity>
+          <linear_acceleration>
+            <!-- m/s^2 | no bias_mean in datasheet -->
+            <x>
+              <xacro:gauss_noise stddev="1.86e-3" bias_mean="1.0e-3" precision="2.40e-3" />
+            </x>
+            <y>
+              <xacro:gauss_noise stddev="1.86e-3" bias_mean="1.0e-3" precision="2.40e-3" />
+            </y>
+            <z>
+              <xacro:gauss_noise stddev="1.86e-3" bias_mean="1.0e-3" precision="2.40e-3" />
+            </z>
+          </linear_acceleration>
+        </imu>
       </sensor>
     </gazebo>

Commit message: Navegación funcionando

File: agro_description/urdf/agro.urdf.xacro (robot description, xacro)
@@ -6,112 +6,13 @@
     <xacro:include filename="$(find agro_description)/urdf/xacro/wheel.xacro"/>
     <xacro:include filename="$(find agro_description)/urdf/xacro/gazebo.xacro"/>
+    <xacro:include filename="$(find agro_description)/urdf/xacro/sensors.xacro"/>
+    <xacro:include filename="$(find agro_description)/urdf/xacro/chassis.xacro"/>
+     <!-- Base footprint-->
     <link name= "base_footprint">
     </link>
-     <!-- Base-->
-    <link name="base_link">
-        <visual>
-            <origin xyz="0.0 0.0 0.0" rpy="0.0 0.0 0.0"/>
-            <geometry>
-                <!--box size="0.5 0.316 0.16"/-->
-                <mesh filename="file://$(find agro_description)/mesh/base.stl" scale="0.001 0.001 0.001"/>
-            </geometry>
-            <material name="wood">
-                <color rgba="0.76 0.60 0.42 1.0"/> <!-- Color madera -->
-            </material>
-        </visual>
-        <xacro:inertial_box mass="${base_mass}" x="${base_largo}" y="${base_ancho}" z="${base_altura}">
-            <origin xyz="0.0 0.0 ${(base_altura)/2}" rpy="0.0 0.0 0.0"/>
-        </xacro:inertial_box>
-        <collision>
-            <origin xyz="0.0 0.0 ${(base_altura)/2}" rpy="0.0 0.0 0.0"/>
-            <geometry>
-                <box size="${base_largo} ${base_ancho} ${base_altura}"/>   <!--0.5 0.316 0.16-->
-            </geometry>
-        </collision>
-    </link>
-    <joint name="base_footprint_joint" type="fixed">
-        <origin xyz="0.0 0.0 0.2" rpy="0.0 0.0 0.0"/>
-        <parent link="base_footprint"/>
-        <child link="base_link"/>
-    </joint>
-    <!-- Chassis-->
-    <link name="chassis_link">
-        <visual>
-            <origin xyz="0.0 0.0 0.0" rpy="0.0 0.0 0.0"/>
-            <geometry>
-                <!--box size="0.5 0.316 0.16"/-->
-                <mesh filename="file://$(find agro_description)/mesh/chassis.stl" scale="0.001 0.001 0.001"/>
-            </geometry>
-            <material name="steel">
-                <color rgba="0.70 0.70 0.70 1.0"/> <!-- Color acero -->
-            </material>
-        </visual>
-        <xacro:inertial_box mass="${chassis_mass}" x="${chassis_largo}" y="${chassis_ancho}" z="${chassis_altura}">
-            <origin xyz="0.0 0.0 ${-(chassis_altura)/2}" rpy="0.0 0.0 0.0"/>
-        </xacro:inertial_box>
-        <collision>
-            <origin xyz="0.0 0.0 ${-(chassis_altura)/2}" rpy="0.0 0.0 0.0"/>
-            <geometry>
-                <box size="${chassis_largo} ${chassis_ancho} ${chassis_altura}"/>
-            </geometry>
-        </collision>
-    </link>
-    <joint name="base_chassis_joint" type="fixed">
-        <origin xyz="0.0 0.0 0.0" rpy="0.0 0.0 0.0"/>
-        <parent link="base_link"/>
-        <child link="chassis_link"/>
-    </joint>
-    <!-- soporte -->
-    <link name="soporte_link">
-        <visual>
-            <origin xyz="0.0 0.0 0.0" rpy="0.0 0.0 0.0"/>
-            <geometry>
-                <mesh filename="file://$(find agro_description)/mesh/soporte.stl" scale="0.001 0.001 0.001"/>
-            </geometry>
-            <material name="steel">
-                <color rgba="0.70 0.70 0.70 1.0"/>
-            </material>
-        </visual>
-        <xacro:inertial_box mass="${soporte_mass}" x="${soporte_largo}" y="${soporte_ancho}" z="${soporte_altura}">
-            <origin xyz="0.0 0.0 0.30" rpy="0.0 0.0 0.0"/>
-        </xacro:inertial_box>
-        <collision>
-            <origin xyz="0.0 0.0 0.30" rpy="0.0 0.0 0.0"/>
-            <geometry>
-                <box size="${soporte_largo} ${soporte_ancho} ${soporte_altura}"/>
-            </geometry>
-        </collision>
-    </link>
-    <joint name="base_soporte_joint" type="fixed">
-        <origin xyz="0.21 0.0 0.16" rpy="0.0 0.0 0.0"/>
-        <parent link="base_link"/>
-        <child link="soporte_link"/>
-    </joint>
-    <!-- base_camara-->
-    <link name="base_camara_link">
-        <visual>
-            <origin xyz="0.0 0.0 0.0" rpy="0.0 0.0 0.0"/>
-            <geometry>
-                <mesh filename="file://$(find agro_description)/mesh/base_camara.stl" scale="0.001 0.001 0.001"/>
-            </geometry>
-            <material name="wood">
-                <color rgba="0.76 0.60 0.42 1.0"/> <!-- Color madera -->
-            </material>
-        </visual>
-        <xacro:inertial_box mass="${base_camara_mass}" x="${base_camara_largo}" y="${base_camara_ancho}" z="${base_camara_altura}">
-            <origin xyz="0.01 0.0 0.0015" rpy="0.0 0.0 0.0"/>
-        </xacro:inertial_box>
-        <collision>
-            <origin xyz="0.01 0.0 0.0015" rpy="0.0 0.0 0.0"/>
-            <geometry>
-                <box size="${base_camara_largo} ${base_camara_ancho} ${base_camara_altura}"/>
-            </geometry>
-        </collision>
-    </link>
-    <joint name="base_camara_joint" type="fixed">
-        <origin xyz="0.21 0.0 0.76" rpy="0.0 0.0 0.0"/>
-        <parent link="base_link"/>
-        <child link="base_camara_link"/>
-    </joint>
+    <!-- Chassis -->
+    <xacro:chassis/>
+    <!-- Soporte -->
+   <xacro:soporte/>
     <!-- Wheels-->
     <xacro:wheel_link prefix="front_left" />
@@ -123,31 +24,13 @@
     <xacro:wheel_joint prefix="near_left" x="-0.210" y="0.224" z="-0.1376"/>
     <xacro:wheel_joint prefix="near_right" x="-0.219" y="-0.224" z="-0.1376"/>
-    <!-- soporte -->
-    <link name="robot_agro/base_footprint/imu_sensor">
-        <visual>
-            <origin xyz="0.0 0.0 0.0" rpy="0.0 0.0 0.0"/>
-            <geometry>
-                <mesh filename="file://$(find agro_description)/mesh/soporte.stl" scale="0.001 0.001 0.001"/>
-            </geometry>
-            <material name="steel">
-                <color rgba="0.70 0.70 0.70 1.0"/>
-            </material>
-        </visual>
-        <xacro:inertial_box mass="${soporte_mass}" x="${soporte_largo}" y="${soporte_ancho}" z="${soporte_altura}">
-            <origin xyz="0.0 0.0 0.30" rpy="0.0 0.0 0.0"/>
-        </xacro:inertial_box>
-        <collision>
-            <origin xyz="0.0 0.0 0.30" rpy="0.0 0.0 0.0"/>
-            <geometry>
-                <box size="${soporte_largo} ${soporte_ancho} ${soporte_altura}"/>
-            </geometry>
-        </collision>
-    </link>
-    <joint name="base_imu_joint" type="fixed">
-        <origin xyz="0.21 0.0 0.16" rpy="0.0 0.0 0.0"/>
-        <parent link="base_footprint"/>
-        <child link="robot_agro/base_footprint/imu_sensor"/>
-    </joint>
+    <!-- camera sensor-->
+    <xacro:camera_sensor/>
+    <!-- imu sensor-->
+    <xacro:imu_sensor/>
+    <!-- lidar sensor-->
+    <xacro:lidar_sensor/>
+    <!-- ros2 control-->
     <xacro:ros2_control/>
+    <!-- gazebo-->
     <xacro:plugins_gazebo/>
 </robot>

File: agro_description/urdf/xacro/gazebo.xacro (robot description, xacro)
@@ -25,25 +25,13 @@
             <xacro:ros2_control wheel="near_left"/>
             <xacro:ros2_control wheel="near_right"/>
-            <sensor name="imu">
-              <state_interface name="orientation.x" />
-              <state_interface name="orientation.y" />
-              <state_interface name="orientation.z" />
-              <state_interface name="orientation.w" />
-              <state_interface name="angular_velocity.x" />
-              <state_interface name="angular_velocity.y" />
-              <state_interface name="angular_velocity.z" />
-              <state_interface name="linear_acceleration.x" />
-              <state_interface name="linear_acceleration.y" />
-              <state_interface name="linear_acceleration.z" />
-            </sensor>
         </ros2_control>
   </xacro:macro>
   <xacro:macro name="plugins_gazebo">
     <gazebo reference="base_footprint">
-        <sensor name="tb3_gps" type="navsat">
+        <sensor name="gps" type="navsat">
           <always_on>true</always_on>
           <update_rate>5</update_rate>
           <pose>0 0 0 0 0 0</pose>
-          <gz_frame_id>base_link</gz_frame_id>
+          <gz_frame_id>base_footprint</gz_frame_id>
           <gps>
             <position_sensing>
@@ -76,5 +64,5 @@
       </noise>
     </xacro:macro>
-    <gazebo reference="base_link">
+    <gazebo reference="imu_link">
       <sensor name="imu_sensor" type="imu">
         <always_on>true</always_on>
@@ -83,4 +71,5 @@
         <visualize>false</visualize>
         <enable_metrics>false</enable_metrics>
+        <gz_frame_id>imu_link</gz_frame_id>
         <imu>
           <angular_velocity>
@@ -112,5 +101,5 @@
     </gazebo>
     <!-- Camera -->
-    <gazebo reference="base_camara_link">
+    <gazebo reference="camera_link">
       <sensor name="camera" type="camera">
           <always_on>1</always_on>
@@ -118,5 +107,36 @@
           <visualize>true</visualize>
           <topic>camera</topic>
-          <frame_id>base_camara_link</frame_id>
+          <gz_frame_id>camera_link</gz_frame_id>
+      </sensor>
+    </gazebo>
+    <gazebo reference="laser_link">
+      <sensor name='gpu_lidar' type='gpu_lidar'>"
+          <topic>scan</topic>
+          <update_rate>20</update_rate>
+          <visualize>true</visualize>
+          <gz_frame_id>laser_link</gz_frame_id>
+          <ray>
+              <scan>
+                  <horizontal>
+                      <samples>640</samples>
+                      <resolution>1</resolution>
+                      <min_angle>-3.096263</min_angle>
+                      <max_angle>3.096263</max_angle>
+                  </horizontal>
+                  <vertical>
+                      <samples>1</samples>
+                      <resolution>0.01</resolution>
+                      <min_angle>0</min_angle>
+                      <max_angle>0</max_angle>
+                  </vertical>
+              </scan>
+              <range>
+                  <min>0.08</min>
+                  <max>10.0</max>
+                  <resolution>0.01</resolution>
+              </range>
+          </ray>
+          <always_on>1</always_on>
+          <visualize>true</visualize>
       </sensor>
     </gazebo>

File: agro_description/urdf/xacro/properties.xacro (robot description, xacro)
@@ -21,3 +21,11 @@
     <xacro:property name="base_camara_ancho" value="0.15" />
     <xacro:property name="base_camara_mass" value="0.05" />
+    <xacro:property name="imu_altura" value="0.02" />
+    <xacro:property name="imu_largo" value="0.02" />
+    <xacro:property name="imu_ancho" value="0.02" />
+    <xacro:property name="imu_mass" value="0.1" />
+    <xacro:property name="lidar_altura" value="0.05" />
+    <xacro:property name="lidar_largo" value="0.05" />
+    <xacro:property name="lidar_ancho" value="0.05" />
+    <xacro:property name="lidar_mass" value="0.1" />
 </robot>
