Commit message: xacro

File: agro_description/urdf/agro.urdf.xacro (robot description, xacro)
@@ -15,4 +15,6 @@
     <!-- Soporte -->
    <xacro:soporte/>
+    <!-- Soporte -->
+   <xacro:head/>
     <!-- Wheels-->
     <xacro:wheel_link prefix="front_left" />
@@ -28,4 +30,6 @@
     <!-- imu sensor-->
     <xacro:imu_sensor/>
+    <!-- gps sensor-->
+    <xacro:gps/>
     <!-- lidar sensor-->
     <xacro:lidar_sensor/>

File: agro_description/urdf/xacro/chassis.xacro (robot description, xacro)
@@ -58,5 +58,5 @@
         </joint>
     </xacro:macro>
-    <!-- Soporte-->
+    <!-- Soporte -->
     <xacro:macro name="soporte">
         <link name="soporte_link">
@@ -86,3 +86,31 @@
         </joint>
     </xacro:macro>
+    <!-- head -->
+    <xacro:macro name="head">
+        <link name="head_link">
+            <visual>
+                <origin xyz="0.0 0.0 0.0" rpy="0.0 0.0 0.0"/>
+                <geometry>
+                    <mesh filename="file://$(find agro_description)/mesh/base_camara.stl" scale="0.001 0.001 0.001"/>
+                </geometry>
+                <material name="wood">
+                    <color rgba="0.76 0.60 0.42 1.0"/> <!-- Color madera -->
+                </material>
+            </visual>
+            <xacro:inertial_box mass="${base_camara_mass}" x="${base_camara_largo}" y="${base_camara_ancho}" z="${base_camara_altura}">
+                <origin xyz="0.01 0.0 0.0015" rpy="0.0 0.0 0.0"/>
+            </xacro:inertial_box>
+            <collision>
+                <origin xyz="0.01 0.0 0.0015" rpy="0.0 0.0 0.0"/>
+                <geometry>
+                    <box size="${base_camara_largo} ${base_camara_ancho} ${base_camara_altura}"/>
+                </geometry>
+            </collision>
+        </link>
+        <joint name="base_head_joint" type="fixed">
+            <origin xyz="0.21 0.0 0.76" rpy="0.0 0.0 0.0"/>
+            <parent link="base_link"/>
+            <child link="head_link"/>
+        </joint>
+    </xacro:macro>
 </robot>

File: agro_description/urdf/xacro/gazebo.xacro (robot description, xacro)
@@ -28,10 +28,11 @@
   </xacro:macro>
   <xacro:macro name="plugins_gazebo">
-    <gazebo reference="base_footprint">
+    <!-- gps base_footprint -->
+    <gazebo reference="gps_link">
         <sensor name="gps" type="navsat">
           <always_on>true</always_on>
           <update_rate>5</update_rate>
           <pose>0 0 0 0 0 0</pose>
-          <gz_frame_id>base_footprint</gz_frame_id>
+          <gz_frame_id>gps_link</gz_frame_id>
           <gps>
             <position_sensing>
@@ -64,4 +65,5 @@
       </noise>
     </xacro:macro>
+    <!-- IMU -->
     <gazebo reference="imu_link">
       <sensor name="imu_sensor" type="imu">
@@ -110,4 +112,5 @@
       </sensor>
     </gazebo>
+    <!-- Laser -->
     <gazebo reference="laser_link">
       <sensor name='gpu_lidar' type='gpu_lidar'>"

File: agro_description/urdf/xacro/properties.xacro (robot description, xacro)
@@ -25,7 +25,15 @@
     <xacro:property name="imu_ancho" value="0.02" />
     <xacro:property name="imu_mass" value="0.1" />
+    <xacro:property name="gps_altura" value="0.02" />
+    <xacro:property name="gps_largo" value="0.02" />
+    <xacro:property name="gps_ancho" value="0.02" />
+    <xacro:property name="gps_mass" value="0.1" />
     <xacro:property name="lidar_altura" value="0.05" />
     <xacro:property name="lidar_largo" value="0.05" />
     <xacro:property name="lidar_ancho" value="0.05" />
     <xacro:property name="lidar_mass" value="0.1" />
+    <xacro:property name="camara_altura" value="0.02" />
+    <xacro:property name="camara_largo" value="0.02" />
+    <xacro:property name="camara_ancho" value="0.02" />
+    <xacro:property name="camara_mass" value="0.1" />
 </robot>

File: agro_description/urdf/xacro/sensors.xacro (robot description, xacro)
@@ -3,17 +3,17 @@
     <xacro:include filename="$(find agro_description)/urdf/xacro/properties.xacro"/>
     <xacro:include filename="$(find agro_description)/urdf/xacro/inertial.xacro"/>
-    <!-- base_camera -->
+    <!-- camera -->
     <xacro:macro name="camera_sensor">
         <link name="camera_link">
-            <visual>
+           <visual>
                 <origin xyz="0.0 0.0 0.0" rpy="0.0 0.0 0.0"/>
                 <geometry>
-                    <mesh filename="file://$(find agro_description)/mesh/base_camara.stl" scale="0.001 0.001 0.001"/>
+                    <box size="${camara_largo} ${camara_ancho} ${camara_altura}"/>
                 </geometry>
-                <material name="wood">
-                    <color rgba="0.76 0.60 0.42 1.0"/> <!-- Color madera -->
+                <material name="red">
+                    <color rgba="0.8 0.0 0.0 1.0"/> <!-- Color madera -->
                 </material>
             </visual>
-            <xacro:inertial_box mass="${base_camara_mass}" x="${base_camara_largo}" y="${base_camara_ancho}" z="${base_camara_altura}">
+            <xacro:inertial_box mass="${camara_mass}" x="${camara_largo}" y="${camara_ancho}" z="${camara_altura}">
                 <origin xyz="0.01 0.0 0.0015" rpy="0.0 0.0 0.0"/>
             </xacro:inertial_box>
@@ -21,10 +21,10 @@
                 <origin xyz="0.01 0.0 0.0015" rpy="0.0 0.0 0.0"/>
                 <geometry>
-                    <box size="${base_camara_largo} ${base_camara_ancho} ${base_camara_altura}"/>
+                    <box size="${camara_largo} ${camara_ancho} ${camara_altura}"/>
                 </geometry>
             </collision>
         </link>
         <joint name="base_camera_joint" type="fixed">
-            <origin xyz="0.21 0.0 0.76" rpy="0.0 0.0 0.0"/>
+            <origin xyz="0.18 0.04 0.77" rpy="0.0 0.0 0.0"/>
             <parent link="base_link"/>
             <child link="camera_link"/>
@@ -39,6 +39,6 @@
                     <box size="${imu_largo} ${imu_ancho} ${imu_altura}"/>
                 </geometry>
-                <material name="wood">
-                    <color rgba="0.76 0.60 0.42 1.0"/> <!-- Color madera -->
+                <material name="black">
+                    <color rgba="0.0 0.0 0.0 1.0"/>
                 </material>
             </visual>
@@ -54,7 +54,35 @@
         </link>
         <joint name="base_imu_joint" type="fixed">
-            <origin xyz="0.0 0.0 0.76" rpy="0.0 0.0 0.0"/>
+            <origin xyz="0.18 0.0 0.015" rpy="0.0 0.0 0.0"/>
             <parent link="base_link"/>
             <child link="imu_link"/>
+        </joint>
+    </xacro:macro>
+    <!-- GPS -->
+    <xacro:macro name="gps">
+        <link name="gps_link">
+            <visual>
+                <origin xyz="0.0 0.0 0.0" rpy="0.0 0.0 0.0"/>
+                <geometry>
+                    <box size="${gps_largo} ${gps_ancho} ${gps_altura}"/>
+                </geometry>
+                <material name="blue">
+                    <color rgba="0.0 0.0 0.8 1.0"/> <!-- Color madera -->
+                </material>
+            </visual>
+            <xacro:inertial_box mass="${gps_mass}" x="${gps_largo}" y="${gps_ancho}" z="${gps_altura}">
+                <origin xyz="0.01 0.0 0.0015" rpy="0.0 0.0 0.0"/>
+            </xacro:inertial_box>
+            <collision>
+                <origin xyz="0.01 0.0 0.0015" rpy="0.0 0.0 0.0"/>
+                <geometry>
+                    <box size="${gps_largo} ${gps_ancho} ${gps_altura}"/>
+                </geometry>
+            </collision>
+        </link>
+        <joint name="base_gps_joint" type="fixed">
+            <origin xyz="0.21 0.0 0.77" rpy="0.0 0.0 0.0"/>
+            <parent link="base_link"/>
+            <child link="gps_link"/>
         </joint>
     </xacro:macro>
@@ -67,6 +95,6 @@
                     <box size="${lidar_largo} ${lidar_ancho} ${lidar_altura}"/>
                 </geometry>
-                <material name="wood">
-                    <color rgba="0.76 0.60 0.42 1.0"/> <!-- Color madera -->
+                <material name="black">
+                    <color rgba="0.0 0.0 0.0 1.0"/> <!-- Color madera -->
                 </material>
             </visual>
@@ -82,5 +110,5 @@
         </link>
         <joint name="base_lidar_joint" type="fixed">
-            <origin xyz="0.0 0.0 0.35" rpy="0.0 0.0 0.0"/>
+            <origin xyz="0.21 0.04 0.185" rpy="0.0 0.0 0.0"/>
             <parent link="base_link"/>
             <child link="laser_link"/>

Commit message: Funcionando

File: agro_description/urdf/agro.urdf.xacro (robot description, xacro)
@@ -15,4 +15,6 @@
     <!-- Soporte -->
    <xacro:soporte/>
+    <!-- Box -->
+   <xacro:box/>
     <!-- Soporte -->
    <xacro:head/>
@@ -38,3 +40,7 @@
     <!-- gazebo-->
     <xacro:plugins_gazebo/>
+    <xacro:wheels_friction side="front_left"/>
+    <xacro:wheels_friction side="front_right"/>
+    <xacro:wheels_friction side="near_left"/>
+    <xacro:wheels_friction side="near_right"/>
 </robot>

File: agro_description/urdf/xacro/chassis.xacro (robot description, xacro)
@@ -114,3 +114,31 @@
         </joint>
     </xacro:macro>
+    <!-- caja equilibrio -->
+    <xacro:macro name="box">
+        <link name="box_link">
+            <visual>
+                <origin xyz="0.0 0.0 0.0" rpy="0.0 0.0 0.0"/>
+                <geometry>
+                    <mesh filename="file://$(find agro_description)/mesh/base_camara.stl" scale="0.001 0.001 0.001"/>
+                </geometry>
+                <material name="wood">
+                    <color rgba="0.76 0.60 0.42 1.0"/> <!-- Color madera -->
+                </material>
+            </visual>
+            <xacro:inertial_box mass="${box_mass}" x="${box_largo}" y="${box_ancho}" z="${box_altura}">
+                <origin xyz="0.01 0.0 0.0015" rpy="0.0 0.0 0.0"/>
+            </xacro:inertial_box>
+            <collision>
+                <origin xyz="0.01 0.0 0.0015" rpy="0.0 0.0 0.0"/>
+                <geometry>
+                    <box size="${box_largo} ${box_ancho} ${box_altura}"/>
+                </geometry>
+            </collision>
+        </link>
+        <joint name="base_box_joint" type="fixed">
+            <origin xyz="-0.21 0.0 0.76" rpy="0.0 0.0 0.0"/>
+            <parent link="base_link"/>
+            <child link="box_link"/>
+        </joint>
+    </xacro:macro>
 </robot>

File: agro_description/urdf/xacro/gazebo.xacro (robot description, xacro)
@@ -27,4 +27,43 @@
         </ros2_control>
   </xacro:macro>
+  <!-- friction wheels -->
+  <xacro:macro name="wheels_friction" params="side">
+    <xacro:if value="${side == 'front_left'}">
+      <xacro:property name="x" value="${wheel_separation_x/2}" />
+      <xacro:property name="y" value="${wheel_separation_y/2}" />
+      <xacro:property name="mesh" value="package://rosbot_xl_description/meshes/${wheel_file}_b.dae" />
+      <xacro:property name="visual_rotation" value="${pi}" />
+      <xacro:property name="fdir" value="1 -1 0" />
+    </xacro:if>
+    <xacro:if value="${side == 'front_right'}">
+      <xacro:property name="x" value="${wheel_separation_x/2}" />
+      <xacro:property name="y" value="${-wheel_separation_y/2}" />
+      <xacro:property name="mesh" value="package://rosbot_xl_description/meshes/${wheel_file}_a.dae" />
+      <xacro:property name="visual_rotation" value="${pi}" />
+      <xacro:property name="fdir" value="1 1 0" />
+    </xacro:if>
+    <xacro:if value="${side == 'near_left'}">
+      <xacro:property name="x" value="${-wheel_separation_x/2}" />
+      <xacro:property name="y" value="${wheel_separation_y/2}" />
+      <xacro:property name="mesh" value="package://rosbot_xl_description/meshes/${wheel_file}_a.dae" />
+      <xacro:property name="visual_rotation" value="${0.0}" />
+      <xacro:property name="fdir" value="1 1 0" />
+    </xacro:if>
+    <xacro:if value="${side == 'near_right'}">
+      <xacro:property name="x" value="${-wheel_separation_x/2}" />
+      <xacro:property name="y" value="${-wheel_separation_y/2}" />
+      <xacro:property name="mesh" value="package://rosbot_xl_description/meshes/${wheel_file}_b.dae" />
+      <xacro:property name="visual_rotation" value="${0.0}" />
+      <xacro:property name="fdir" value="1 -1 0" />
+    </xacro:if>
+      <gazebo reference="${side}_wheel_link">
+            <kp>1000000.0</kp>
+            <kd>50</kd>
+            <mu1>100</mu1>
+            <mu2>100</mu2>
+            <minDepth>0.02</minDepth>
+            <implicitSpringDamper>1</implicitSpringDamper>
+      </gazebo>
+  </xacro:macro >
   <xacro:macro name="plugins_gazebo">
     <!-- gps base_footprint -->
@@ -106,6 +145,6 @@
       <sensor name="camera" type="camera">
           <always_on>1</always_on>
-          <update_rate>30</update_rate>
-          <visualize>true</visualize>
+          <update_rate>20</update_rate>
+          <visualize>false</visualize>
           <topic>camera</topic>
           <gz_frame_id>camera_link</gz_frame_id>
@@ -147,5 +186,5 @@
               <range>
                   <min>0.08</min>
-                  <max>10.0</max>
+                  <max>50.0</max>
                   <resolution>0.01</resolution>
               </range>

File: agro_description/urdf/xacro/properties.xacro (robot description, xacro)
@@ -4,5 +4,5 @@
     <xacro:property name="wheel_radius" value="0.0601" />
     <xacro:property name="wheel_length" value="0.0615" />
-    <xacro:property name="wheel_mass" value="0.2" />
+    <xacro:property name="wheel_mass" value="0.4" />
     <xacro:property name="base_altura" value="0.16" />
     <xacro:property name="base_largo" value="0.5" />
@@ -12,5 +12,5 @@
     <xacro:property name="chassis_largo" value="0.46" />
     <xacro:property name="chassis_ancho" value="0.44" />
-    <xacro:property name="chassis_mass" value="0.2" />
+    <xacro:property name="chassis_mass" value="2.0" />
     <xacro:property name="soporte_altura" value="0.6" />
     <xacro:property name="soporte_largo" value="0.02" />
@@ -24,16 +24,20 @@
     <xacro:property name="imu_largo" value="0.02" />
     <xacro:property name="imu_ancho" value="0.02" />
-    <xacro:property name="imu_mass" value="0.1" />
+    <xacro:property name="imu_mass" value="0.001" />
     <xacro:property name="gps_altura" value="0.02" />
     <xacro:property name="gps_largo" value="0.02" />
     <xacro:property name="gps_ancho" value="0.02" />
-    <xacro:property name="gps_mass" value="0.1" />
+    <xacro:property name="gps_mass" value="0.001" />
     <xacro:property name="lidar_altura" value="0.05" />
     <xacro:property name="lidar_largo" value="0.05" />
     <xacro:property name="lidar_ancho" value="0.05" />
-    <xacro:property name="lidar_mass" value="0.1" />
+    <xacro:property name="lidar_mass" value="0.001" />
+    <xacro:property name="box_altura" value="0.2" />
+    <xacro:property name="box_largo" value="0.02" />
+    <xacro:property name="box_ancho" value="0.02" />
+    <xacro:property name="box_mass" value="0.3" />
     <xacro:property name="camara_altura" value="0.02" />
     <xacro:property name="camara_largo" value="0.02" />
     <xacro:property name="camara_ancho" value="0.02" />
-    <xacro:property name="camara_mass" value="0.1" />
+    <xacro:property name="camara_mass" value="0.001" />
 </robot>

Commit message: Se volvio a la versiond e gazebo

File: agro_description/urdf/agro.urdf.xacro (robot description, xacro)
@@ -16,5 +16,5 @@
    <xacro:soporte/>
     <!-- Box -->
-   <xacro:box/>
+   <!--xacro:box/-->
     <!-- Soporte -->
    <xacro:head/>
@@ -40,7 +40,7 @@
     <!-- gazebo-->
     <xacro:plugins_gazebo/>
-    <xacro:wheels_friction side="front_left"/>
+    <!--xacro:wheels_friction side="front_left"/>
     <xacro:wheels_friction side="front_right"/>
     <xacro:wheels_friction side="near_left"/>
-    <xacro:wheels_friction side="near_right"/>
+    <xacro:wheels_friction side="near_right"/-->
 </robot>

File: agro_description/urdf/xacro/chassis.xacro (robot description, xacro)
@@ -17,5 +17,6 @@
             </visual>
             <xacro:inertial_box mass="${base_mass}" x="${base_largo}" y="${base_ancho}" z="${base_altura}">
-                <origin xyz="0.0 0.0 ${(base_altura)/2}" rpy="0.0 0.0 0.0"/>
+                <!--origin xyz="0.0 0.0 ${(base_altura)/2}" rpy="0.0 0.0 0.0"/-->
+                <origin xyz="0.0 0.0 0.0" rpy="0.0 0.0 0.0"/>
             </xacro:inertial_box>
             <collision>
@@ -43,5 +44,6 @@
             </visual>
             <xacro:inertial_box mass="${chassis_mass}" x="${chassis_largo}" y="${chassis_ancho}" z="${chassis_altura}">
-                <origin xyz="0.0 0.0 ${-(chassis_altura)/2}" rpy="0.0 0.0 0.0"/>
+                <!--origin xyz="0.0 0.0 ${-(chassis_altura)/2}" rpy="0.0 0.0 0.0"/-->
+                <origin xyz="0.0 0.0 0.0" rpy="0.0 0.0 0.0"/>
             </xacro:inertial_box>
             <collision>
