Commit message: vision

File: agro_description/urdf/xacro/sensors.xacro (robot description, xacro)
@@ -26,5 +26,5 @@
         </link>
         <joint name="base_camera_joint" type="fixed">
-            <origin xyz="0.18 0.04 0.77" rpy="0.0 0.0 0.0"/>
+            <origin xyz="0.18 0.06 0.77" rpy="0.0 0.0 0.0"/>
             <parent link="base_link"/>
             <child link="camera_link"/>

Commit message: camara

File: agro_description/urdf/xacro/sensors.xacro (robot description, xacro)
@@ -26,5 +26,5 @@
         </link>
         <joint name="base_camera_joint" type="fixed">
-            <origin xyz="0.18 0.06 0.77" rpy="0.0 0.0 0.0"/>
+            <origin xyz="0.18 0.08 0.77" rpy="0.0 0.0 0.0"/>
             <parent link="base_link"/>
             <child link="camera_link"/>

Commit message: remaping

File: agro_description/urdf/xacro/sensors.xacro (robot description, xacro)
@@ -26,5 +26,5 @@
         </link>
         <joint name="base_camera_joint" type="fixed">
-            <origin xyz="0.18 0.08 0.77" rpy="0.0 0.0 0.0"/>
+            <origin xyz="0.18 0.08 0.40" rpy="0.0 0.0 1.57079632679"/>
             <parent link="base_link"/>
             <child link="camera_link"/>
